Commit message: The Back Leg

File: body.urdf (robot description, URDF)
Before this commit: robot robot, 3 links, 2 joints
Links:
- link BackLeg: geometry collision box size=0.2 1.0 0.2; visual box size=0.2 1.0 0.2
Joints:
- joint Torso_BackLeg: origin xyz=1 0 1 rpy=0 0 0 -> xyz=0 -0.5 1 rpy=0 0 0

Commit message: Jk now finished left and right legs

File: body.urdf (robot description, URDF)
Before this commit: robot robot, 3 links, 2 joints
Links:
- added link LeftLeg, mass 1; collision box size=1.0 0.2 0.2; visual box size=1.0 0.2 0.2
- added link RightLeg, mass 1; collision box size=1.0 0.2 0.2; visual box size=1.0 0.2 0.2
Joints:
- added joint Torso_LeftLeg: type revolute, parent Torso, child LeftLeg, origin xyz=-0.5 0 1 rpy=0 0 0, axis 0 1 0, limit lower=-3.14159 upper=3.14159 effort=0.0 velocity=0.0
- added joint Torso_RightLeg: type revolute, parent Torso, child RightLeg, origin xyz=0.5 0 1 rpy=0 0 0, axis 0 1 0, limit lower=-3.14159 upper=3.14159 effort=0.0 velocity=0.0

Commit message: somewhat working final project

File: body.urdf (robot description, URDF)
Before this commit: robot robot, 9 links, 8 joints
Links:
- removed link BackLeg
- removed link BackLowerLeg
- removed link FrontLeg
- removed link FrontLowerLeg
- added link LeftFoot, mass 1; collision box size=1.0 0.5 0.5; visual box size=1.0 0.5 0.5
- added link RightFoot, mass 1; collision box size=1.0 0.5 0.5; visual box size=1.0 0.5 0.5
- link LeftLeg: geometry collision box size=0.2 0.2 1.0; visual box size=0.2 0.2 1.0
- link RightLeg: geometry collision box size=0.2 0.2 1.0; visual box size=0.2 0.2 1.0
Joints:
- removed joint BackLeg_BackLowerLeg
- removed joint FrontLeg_FrontLowerLeg
- removed joint Torso_BackLeg
- removed joint Torso_FrontLeg
- added joint LeftLowerLeg_LeftFoot: type revolute, parent LeftLowerLeg, child LeftFoot, origin xyz=0 0 -1 rpy=0 0 0, axis 0 1 0, limit lower=-3.14159 upper=3.14159 effort=0.0 velocity=0.0
- added joint RightLowerLeg_RightFoot: type revolute, parent RightLowerLeg, child RightFoot, origin xyz=0 0 -1.0 rpy=0 0 0, axis 0 1 0, limit lower=-3.14159 upper=3.14159 effort=0.0 velocity=0.0
- joint LeftLeg_LeftLowerLeg: origin xyz=-1 0 0 rpy=0 0 0 -> xyz=0 0 -1 rpy=0 0 0
- joint RightLeg_RightLowerLeg: origin xyz=1 0 0 rpy=0 0 0 -> xyz=0 0 -1.0 rpy=0 0 0
- joint Torso_LeftLeg: origin xyz=-0.5 0 1 rpy=0 0 0 -> xyz=0 -0.5 2.5 rpy=0 0 0
- joint Torso_RightLeg: origin xyz=0.5 0 1 rpy=0 0 0 -> xyz=0 0.5 2.5 rpy=0 0 0

Commit message: Finished 3D morphos

File: body.urdf (robot description, URDF)
Before this commit: robot robot, 7 links, 6 joints
Links:
- removed link LeftFoot
- removed link LeftLeg
- removed link LeftLowerLeg
- removed link RightFoot
- removed link RightLeg
- removed link RightLowerLeg
- removed link Torso
- added link Head, mass 1; collision box size=0.99330110665343 0.14020201586286585 0.24133334006402363; visual box size=0.99330110665343 0.14020201586286585 0.24133334006402363
- added link Link-x10, mass 1; collision box size=0.2630061141777216 0.628216471847177 0.9290785088531935; visual box size=0.2630061141777216 0.628216471847177 0.9290785088531935
- added link Link-x11, mass 1; collision box size=0.9837371863780355 0.049756810162816856 0.06413085067861901; visual box size=0.9837371863780355 0.049756810162816856 0.06413085067861901
- added link Link-x2, mass 1; collision box size=0.5469485799619188 0.4338040993642286 0.7558102700653434; visual box size=0.5469485799619188 0.4338040993642286 0.7558102700653434
- added link Link-x3, mass 1; collision box size=0.327287876836471 0.624382644366813 0.35303816795585485; visual box size=0.327287876836471 0.624382644366813 0.35303816795585485
- added link Link-x6, mass 1; collision box size=0.7843907484774278 0.7854457864055909 0.13486742031424537; visual box size=0.7843907484774278 0.7854457864055909 0.13486742031424537
- added link Link-x7, mass 1; collision box size=0.14172649862361053 0.41452856475741695 0.33540578734306536; visual box size=0.14172649862361053 0.41452856475741695 0.33540578734306536
- added link Link-x8, mass 1; collision box size=0.6563962852173223 0.9300168687993656 0.7138032372521665; visual box size=0.6563962852173223 0.9300168687993656 0.7138032372521665
- added link Link-y1, mass 1; collision box size=0.8265274659270198 0.43458762180995003 0.008834826308734889; visual box size=0.8265274659270198 0.43458762180995003 0.008834826308734889
- added link Link-y5, mass 1; collision box size=0.039424577975163966 0.7460555279532477 0.48927452364249313; visual box size=0.039424577975163966 0.7460555279532477 0.48927452364249313
- added link Link-y9, mass 1; collision box size=0.602690853396696 0.5757368070877635 0.49614004487955676; visual box size=0.602690853396696 0.5757368070877635 0.49614004487955676
- added link Link-z4, mass 1; collision box size=0.7509867933404144 0.9067520904515937 0.5605694603741277; visual box size=0.7509867933404144 0.9067520904515937 0.5605694603741277
Joints:
- removed joint LeftLeg_LeftLowerLeg
- removed joint LeftLowerLeg_LeftFoot
- removed joint RightLeg_RightLowerLeg
- removed joint RightLowerLeg_RightFoot
- removed joint Torso_LeftLeg
- removed joint Torso_RightLeg
- added joint Head_Link-y1: type revolute, parent Head, child Link-y1, origin xyz=0 0.07010100793143292 0.9290785088531935 rpy=0 0 0, axis 0 0 1, limit lower=-3.14159 upper=3.14159 effort=0.0 velocity=0.0
- added joint Link-x10_Link-x11: type revolute, parent Link-x10, child Link-x11, origin xyz=0.2630061141777216 0 0 rpy=0 0 0, axis 0 1 1, limit lower=-3.14159 upper=3.14159 effort=0.0 velocity=0.0
- added joint Link-x2_Link-x3: type revolute, parent Link-x2, child Link-x3, origin xyz=0.5469485799619188 0 0 rpy=0 0 0, axis 0 1 1, limit lower=-3.14159 upper=3.14159 effort=0.0 velocity=0.0
- added joint Link-x3_Link-z4: type revolute, parent Link-x3, child Link-z4, origin xyz=0.1636439384182355 0 0.17651908397792743 rpy=0 0 0, axis 0 1 0, limit lower=-3.14159 upper=3.14159 effort=0.0 velocity=0.0
- added joint Link-x6_Link-x7: type revolute, parent Link-x6, child Link-x7, origin xyz=0.7843907484774278 0 0 rpy=0 0 0, axis 0 1 1, limit lower=-3.14159 upper=3.14159 effort=0.0 velocity=0.0
- added joint Link-x7_Link-x8: type revolute, parent Link-x7, child Link-x8, origin xyz=0.14172649862361053 0 0 rpy=0 0 0, axis 0 1 1, limit lower=-3.14159 upper=3.14159 effort=0.0 velocity=0.0
- added joint Link-x8_Link-y9: type revolute, parent Link-x8, child Link-y9, origin xyz=0.32819814260866115 0.4650084343996828 0 rpy=0 0 0, axis 0 0 1, limit lower=-3.14159 upper=3.14159 effort=0.0 velocity=0.0
- added joint Link-y1_Link-x2: type revolute, parent Link-y1, child Link-x2, origin xyz=0.4132637329635099 0.21729381090497502 0 rpy=0 0 0, axis 0 0 1, limit lower=-3.14159 upper=3.14159 effort=0.0 velocity=0.0
- added joint Link-y5_Link-x6: type revolute, parent Link-y5, child Link-x6, origin xyz=0.019712288987581983 0.37302776397662385 0 rpy=0 0 0, axis 0 0 1, limit lower=-3.14159 upper=3.14159 effort=0.0 velocity=0.0
- added joint Link-y9_Link-x10: type revolute, parent Link-y9, child Link-x10, origin xyz=0.301345426698348 0.28786840354388177 0 rpy=0 0 0, axis 0 0 1, limit lower=-3.14159 upper=3.14159 effort=0.0 velocity=0.0
- added joint Link-z4_Link-y5: type revolute, parent Link-z4, child Link-y5, origin xyz=0 0.45337604522579683 0.28028473018706385 rpy=0 0 0, axis 1 0 0, limit lower=-3.14159 upper=3.14159 effort=0.0 velocity=0.0

Commit message: Somewhat 3d morph

File: body.urdf (robot description, URDF)
Before this commit: robot robot, 12 links, 11 joints
Links:
- removed link Head
- removed link Link-x10
- removed link Link-x2
- removed link Link-x3
- removed link Link-x7
- removed link Link-x8
- removed link Link-y5
- removed link Link-y9
- removed link Link-z4
- added link Link-x0, mass 1; collision box size=0.5696283126898227 0.5548721456207658 0.42642605154915547; visual box size=0.5696283126898227 0.5548721456207658 0.42642605154915547
- added link Link-x15, mass 1; collision box size=0.3622996183521665 0.12501299355768158 0.16132089934942773; visual box size=0.3622996183521665 0.12501299355768158 0.16132089934942773
- added link Link-x18, mass 1; collision box size=0.5486137627163392 0.024240001285998236 0.7529571338706489; visual box size=0.5486137627163392 0.024240001285998236 0.7529571338706489
- added link Link-x19, mass 1; collision box size=0.3508975965428871 0.6999687046979262 0.2503686158240339; visual box size=0.3508975965428871 0.6999687046979262 0.2503686158240339
- added link Link-x21, mass 1; collision box size=0.37116251624394736 0.5053576217669303 0.5440472679777312; visual box size=0.37116251624394736 0.5053576217669303 0.5440472679777312
- added link Link-x9, mass 1; collision box size=0.9494780169775451 0.7423561657921315 0.849053427115123; visual box size=0.9494780169775451 0.7423561657921315 0.849053427115123
- added link Link-y13, mass 1; collision box size=0.06810879402524983 0.8382546256467166 0.3558559322035644; visual box size=0.06810879402524983 0.8382546256467166 0.3558559322035644
- added link Link-y14, mass 1; collision box size=0.33929821981499886 0.06876369098409141 0.9506353530634845; visual box size=0.33929821981499886 0.06876369098409141 0.9506353530634845
- added link Link-y16, mass 1; collision box size=0.949210936239449 0.4219578195697433 0.8442057104574648; visual box size=0.949210936239449 0.4219578195697433 0.8442057104574648
- added link Link-y20, mass 1; collision box size=0.5311507546703057 0.5936930246261156 0.1743561825300276; visual box size=0.5311507546703057 0.5936930246261156 0.1743561825300276
- added link Link-y23, mass 1; collision box size=0.24221104502665358 0.21036026738187352 0.23568724104492578; visual box size=0.24221104502665358 0.21036026738187352 0.23568724104492578
- added link Link-y4, mass 1; collision box size=0.7325582635196397 0.9245101206180499 0.17338769987377312; visual box size=0.7325582635196397 0.9245101206180499 0.17338769987377312
- added link Link-y7, mass 1; collision box size=0.16708402804542455 0.7744974679674835 0.33104003768466195; visual box size=0.16708402804542455 0.7744974679674835 0.33104003768466195
- added link Link-z10, mass 1; collision box size=0.6336426328948055 0.34727283422448074 0.44119383845070426; visual box size=0.6336426328948055 0.34727283422448074 0.44119383845070426
- added link Link-z12, mass 1; collision box size=0.044710857575020024 0.6679474923066937 0.14871455408691292; visual box size=0.044710857575020024 0.6679474923066937 0.14871455408691292
- added link Link-z17, mass 1; collision box size=0.9634351837940563 0.3502922188434038 0.6810193748946952; visual box size=0.9634351837940563 0.3502922188434038 0.6810193748946952
- added link Link-z2, mass 1; collision box size=0.20858039933341477 0.9068326618172867 0.21888143236597601; visual box size=0.20858039933341477 0.9068326618172867 0.21888143236597601
- added link Link-z22, mass 1; collision box size=0.25068524072935316 0.174458572110593 0.8813575749933087; visual box size=0.25068524072935316 0.174458572110593 0.8813575749933087
- added link Link-z3, mass 1; collision box size=0.1613949713986117 0.014068092202585536 0.23265164655605464; visual box size=0.1613949713986117 0.014068092202585536 0.23265164655605464
- added link Link-z5, mass 1; collision box size=0.8687748541140948 0.3127628690463611 0.2740223067613603; visual box size=0.8687748541140948 0.3127628690463611 0.2740223067613603
- added link Link-z8, mass 1; collision box size=0.18479218389306062 0.10380400104823828 0.47583699149148473; visual box size=0.18479218389306062 0.10380400104823828 0.47583699149148473
- link Link-x11: geometry collision box size=0.9280280257567504 0.8740947034255337 0.04179037594910584; visual box size=0.9280280257567504 0.8740947034255337 0.04179037594910584
- link Link-x6: geometry collision box size=0.4144959037070409 0.5451223867975967 0.46471290348039884; visual box size=0.4144959037070409 0.5451223867975967 0.46471290348039884
- link Link-y1: geometry collision box size=0.055365426836538334 0.47221468690510293 0.4507097757280426; visual box size=0.055365426836538334 0.47221468690510293 0.4507097757280426
Joints:
- removed joint Head_Link-y1
- removed joint Link-x10_Link-x11
- removed joint Link-x2_Link-x3
- removed joint Link-x3_Link-z4
- removed joint Link-x6_Link-x7
- removed joint Link-x7_Link-x8
- removed joint Link-x8_Link-y9
- removed joint Link-y1_Link-x2
- removed joint Link-y5_Link-x6
- removed joint Link-y9_Link-x10
- removed joint Link-z4_Link-y5
- added joint Link-x0_Link-y1: type revolute, parent Link-x0, child Link-y1, origin xyz=0 0.2774360728103829 0.9994474958213642 rpy=0 0 0, axis 0 0 1, limit lower=-3.14159 upper=3.14159 effort=0.0 velocity=0.0
- added joint Link-x0_Link-z2: type revolute, parent Link-x0, child Link-z2, origin xyz=0 0 1.2126605215959418 rpy=0 0 0, axis 1 1 0, limit lower=-3.14159 upper=3.14159 effort=0.0 velocity=0.0
- added joint Link-x6_Link-x9: type revolute, parent Link-x6, child Link-x9, origin xyz=0.4144959037070409 0 0 rpy=0 0 0, axis 0 1 1, limit lower=-3.14159 upper=3.14159 effort=0.0 velocity=0.0
- added joint Link-x6_Link-y7: type revolute, parent Link-x6, child Link-y7, origin xyz=0.20724795185352046 0.27256119339879836 0 rpy=0 0 0, axis 0 0 1, limit lower=-3.14159 upper=3.14159 effort=0.0 velocity=0.0
- added joint Link-x6_Link-z8: type revolute, parent Link-x6, child Link-z8, origin xyz=0.20724795185352046 0 0.23235645174019942 rpy=0 0 0, axis 0 1 0, limit lower=-3.14159 upper=3.14159 effort=0.0 velocity=0.0
- added joint Link-x9_Link-y14: type revolute, parent Link-x9, child Link-y14, origin xyz=0.47473900848877254 0.37117808289606574 0 rpy=0 0 0, axis 0 0 1, limit lower=-3.14159 upper=3.14159 effort=0.0 velocity=0.0
- added joint Link-y14_Link-x15: type revolute, parent Link-y14, child Link-x15, origin xyz=0.16964910990749943 0.034381845492045704 0 rpy=0 0 0, axis 0 0 1, limit lower=-3.14159 upper=3.14159 effort=0.0 velocity=0.0
- added joint Link-y1_Link-z10: type revolute, parent Link-y1, child Link-z10, origin xyz=0 0.23610734345255147 0.2253548878640213 rpy=0 0 0, axis 1 0 0, limit lower=-3.14159 upper=3.14159 effort=0.0 velocity=0.0
- added joint Link-y20_Link-x21: type revolute, parent Link-y20, child Link-x21, origin xyz=0.26557537733515285 0.2968465123130578 0 rpy=0 0 0, axis 0 0 1, limit lower=-3.14159 upper=3.14159 effort=0.0 velocity=0.0
- added joint Link-y20_Link-y23: type revolute, parent Link-y20, child Link-y23, origin xyz=0 0.5936930246261156 0 rpy=0 0 0, axis 1 0 1, limit lower=-3.14159 upper=3.14159 effort=0.0 velocity=0.0
- added joint Link-y20_Link-z22: type revolute, parent Link-y20, child Link-z22, origin xyz=0 0.2968465123130578 0.0871780912650138 rpy=0 0 0, axis 1 0 0, limit lower=-3.14159 upper=3.14159 effort=0.0 velocity=0.0
- added joint Link-y4_Link-x11: type revolute, parent Link-y4, child Link-x11, origin xyz=0.36627913175981985 0.46225506030902497 0 rpy=0 0 0, axis 0 0 1, limit lower=-3.14159 upper=3.14159 effort=0.0 velocity=0.0
- added joint Link-y4_Link-y13: type revolute, parent Link-y4, child Link-y13, origin xyz=0 0.9245101206180499 0 rpy=0 0 0, axis 1 0 1, limit lower=-3.14159 upper=3.14159 effort=0.0 velocity=0.0
- added joint Link-y4_Link-z12: type revolute, parent Link-y4, child Link-z12, origin xyz=0 0.46225506030902497 0.08669384993688656 rpy=0 0 0, axis 1 0 0, limit lower=-3.14159 upper=3.14159 effort=0.0 velocity=0.0
- added joint Link-y7_Link-x18: type revolute, parent Link-y7, child Link-x18, origin xyz=0.08354201402271227 0.38724873398374177 0 rpy=0 0 0, axis 0 0 1, limit lower=-3.14159 upper=3.14159 effort=0.0 velocity=0.0
- added joint Link-y7_Link-y16: type revolute, parent Link-y7, child Link-y16, origin xyz=0 0.7744974679674835 0 rpy=0 0 0, axis 1 0 1, limit lower=-3.14159 upper=3.14159 effort=0.0 velocity=0.0
- added joint Link-y7_Link-z17: type revolute, parent Link-y7, child Link-z17, origin xyz=0 0.38724873398374177 0.16552001884233097 rpy=0 0 0, axis 1 0 0, limit lower=-3.14159 upper=3.14159 effort=0.0 velocity=0.0
- added joint Link-z10_Link-x19: type revolute, parent Link-z10, child Link-x19, origin xyz=0.31682131644740275 0 0.22059691922535213 rpy=0 0 0, axis 0 1 0, limit lower=-3.14159 upper=3.14159 effort=0.0 velocity=0.0
- added joint Link-z10_Link-y20: type revolute, parent Link-z10, child Link-y20, origin xyz=0 0.17363641711224037 0.22059691922535213 rpy=0 0 0, axis 1 0 0, limit lower=-3.14159 upper=3.14159 effort=0.0 velocity=0.0
- added joint Link-z2_Link-y4: type revolute, parent Link-z2, child Link-y4, origin xyz=0 0.45341633090864336 0.10944071618298801 rpy=0 0 0, axis 1 0 0, limit lower=-3.14159 upper=3.14159 effort=0.0 velocity=0.0
- added joint Link-z2_Link-z3: type revolute, parent Link-z2, child Link-z3, origin xyz=0 0 0.21888143236597601 rpy=0 0 0, axis 1 1 0, limit lower=-3.14159 upper=3.14159 effort=0.0 velocity=0.0
- added joint Link-z3_Link-x6: type revolute, parent Link-z3, child Link-x6, origin xyz=0.08069748569930585 0 0.11632582327802732 rpy=0 0 0, axis 0 1 0, limit lower=-3.14159 upper=3.14159 effort=0.0 velocity=0.0
- added joint Link-z3_Link-z5: type revolute, parent Link-z3, child Link-z5, origin xyz=0 0 0.23265164655605464 rpy=0 0 0, axis 1 1 0, limit lower=-3.14159 upper=3.14159 effort=0.0 velocity=0.0

Commit message: I Think I've finished the Robot but limbs overlap

File: body.urdf (robot description, URDF)
Before this commit: robot robot, 24 links, 23 joints
Links:
- removed link Link-x11
- removed link Link-x15
- removed link Link-x18
- removed link Link-x19
- removed link Link-x21
- removed link Link-x6
- removed link Link-x9
- removed link Link-y1
- removed link Link-y13
- removed link Link-y14
- removed link Link-y16
- removed link Link-y20
- removed link Link-y23
- removed link Link-y4
- removed link Link-y7
- removed link Link-z10
- removed link Link-z12
- removed link Link-z17
- removed link Link-z2
- removed link Link-z22
- removed link Link-z3
- removed link Link-z5
- removed link Link-z8
- added link Link-x2, mass 1; collision box size=0.0629166354899462 0.8548062895720026 0.5954286605739336; visual box size=0.0629166354899462 0.8548062895720026 0.5954286605739336
- added link Link-y3, mass 1; collision box size=0.151914638725962 0.5099502569863811 0.6237127179144237; visual box size=0.151914638725962 0.5099502569863811 0.6237127179144237
- added link Link-y5, mass 1; collision box size=0.01078952257438337 0.8436302414489311 0.7840452055685069; visual box size=0.01078952257438337 0.8436302414489311 0.7840452055685069
- added link Link-z1, mass 1; collision box size=0.18275930546249253 0.22124138796233428 0.4292750243493524; visual box size=0.18275930546249253 0.22124138796233428 0.4292750243493524
- added link Link-z4, mass 1; collision box size=0.06454820168397479 0.1809120781781235 0.41588895176791574; visual box size=0.06454820168397479 0.1809120781781235 0.41588895176791574
- added link Link-z6, mass 1; collision box size=0.20257320978890958 0.9472793471637014 0.5257907102993518; visual box size=0.20257320978890958 0.9472793471637014 0.5257907102993518
- link Link-x0: geometry collision box size=0.8169373613746115 0.4246761914937198 0.714440780299139; visual box size=0.8169373613746115 0.4246761914937198 0.714440780299139
Joints:
- removed joint Link-x0_Link-y1
- removed joint Link-x0_Link-z2
- removed joint Link-x6_Link-x9
- removed joint Link-x6_Link-y7
- removed joint Link-x6_Link-z8
- removed joint Link-x9_Link-y14
- removed joint Link-y14_Link-x15
- removed joint Link-y1_Link-z10
- removed joint Link-y20_Link-x21
- removed joint Link-y20_Link-y23
- removed joint Link-y20_Link-z22
- removed joint Link-y4_Link-x11
- removed joint Link-y4_Link-y13
- removed joint Link-y4_Link-z12
- removed joint Link-y7_Link-x18
- removed joint Link-y7_Link-y16
- removed joint Link-y7_Link-z17
- removed joint Link-z10_Link-x19
- removed joint Link-z10_Link-y20
- removed joint Link-z2_Link-y4
- removed joint Link-z2_Link-z3
- removed joint Link-z3_Link-x6
- removed joint Link-z3_Link-z5
- added joint Link-x0_Link-z1: type revolute, parent Link-x0, child Link-z1, origin xyz=0 0 1.357136196169094 rpy=0 0 0, axis 0 0 1, limit lower=-3.14159 upper=3.14159 effort=0.0 velocity=0.0
- added joint Link-z1_Link-x2: type revolute, parent Link-z1, child Link-x2, origin xyz=0.4154857200072506 0 0 rpy=0 0 0, axis 1 0 0, limit lower=-3.14159 upper=3.14159 effort=0.0 velocity=0.0
- added joint Link-z1_Link-y3: type revolute, parent Link-z1, child Link-y3, origin xyz=0 0.13775113243670017 0 rpy=0 0 0, axis 0 1 0, limit lower=-3.14159 upper=3.14159 effort=0.0 velocity=0.0
- added joint Link-z1_Link-z4: type revolute, parent Link-z1, child Link-z4, origin xyz=0 0 0.4292750243493524 rpy=0 0 0, axis 0 0 1, limit lower=-3.14159 upper=3.14159 effort=0.0 velocity=0.0
- added joint Link-z4_Link-y5: type revolute, parent Link-z4, child Link-y5, origin xyz=0 0.040686337673459194 0 rpy=0 0 0, axis 0 1 0, limit lower=-3.14159 upper=3.14159 effort=0.0 velocity=0.0
- added joint Link-z4_Link-z6: type revolute, parent Link-z4, child Link-z6, origin xyz=0 0 0.41588895176791574 rpy=0 0 0, axis 0 0 1, limit lower=-3.14159 upper=3.14159 effort=0.0 velocity=0.0
