Commit message: Finished Overlapping Robot

File: body.urdf (robot description, URDF)
Before this commit: robot robot, 7 links, 6 joints
Links:
- removed link Link-y5
- removed link Link-z6
- added link Link-z5, mass 1; collision box size=0.7769734266057364 0.827886902774269 0.15448035132713955; visual box size=0.7769734266057364 0.827886902774269 0.15448035132713955
- link Link-x0: geometry collision box size=0.5188064762652517 0.9589082011404115 0.8096606811726296; visual box size=0.5188064762652517 0.9589082011404115 0.8096606811726296
- link Link-x2: geometry collision box size=0.5100324289481527 0.5917958303148464 0.7632447362363; visual box size=0.5100324289481527 0.5917958303148464 0.7632447362363
- link Link-y3: geometry collision box size=0.08373874056435482 0.6081876885055766 0.39312140521446376; visual box size=0.08373874056435482 0.6081876885055766 0.39312140521446376
- link Link-z1: geometry collision box size=0.9075668623485278 0.07003450525794896 0.1556249959011159; visual box size=0.9075668623485278 0.07003450525794896 0.1556249959011159
- link Link-z4: geometry collision box size=0.7093930205900036 0.2135669500635809 0.42219752139105876; visual box size=0.7093930205900036 0.2135669500635809 0.42219752139105876
Joints:
- removed joint Link-z1_Link-x2
- removed joint Link-z1_Link-y3
- removed joint Link-z1_Link-z4
- removed joint Link-z4_Link-y5
- removed joint Link-z4_Link-z6
- added joint Link-x0_Link-x2: type revolute, parent Link-x0, child Link-x2, origin xyz=0.25940323813262584 0 0.8096606811726296 rpy=0 0 0, axis 0 0 1, limit lower=-3.14159 upper=3.14159 effort=0.0 velocity=0.0
- added joint Link-x2_Link-y3: type revolute, parent Link-x2, child Link-y3, origin xyz=0 0.2958979151574232 0 rpy=0 0 0, axis 0 0 1, limit lower=-3.14159 upper=3.14159 effort=0.0 velocity=0.0
- added joint Link-x2_Link-z4: type revolute, parent Link-x2, child Link-z4, origin xyz=0 0 0.38162236811815 rpy=0 0 0, axis 1 0 0, limit lower=-3.14159 upper=3.14159 effort=0.0 velocity=0.0
- added joint Link-z4_Link-z5: type revolute, parent Link-z4, child Link-z5, origin xyz=0 0 0.42219752139105876 rpy=0 0 0, axis 1 0 0, limit lower=-3.14159 upper=3.14159 effort=0.0 velocity=0.0
- joint Link-x0_Link-z1: axis 0 0 1 -> 1 0 0; origin xyz=0 0 1.357136196169094 rpy=0 0 0 -> xyz=0 0 1.2144910217589444 rpy=0 0 0

Commit message: Somewhat working but with intersections :/

File: body.urdf (robot description, URDF)
Before this commit: robot robot, 4 links, 3 joints
Links:
- removed link Link-x1
- removed link Link-z2
- added link Link-x2, mass 1; collision box size=0.867184041678314 0.26513307180416035 0.6557069163228023; visual box size=0.867184041678314 0.26513307180416035 0.6557069163228023
- added link Link-y1, mass 1; collision box size=0.6675601674807339 0.4829636587960703 0.7053158690670012; visual box size=0.6675601674807339 0.4829636587960703 0.7053158690670012
- added link Link-y5, mass 1; collision box size=0.5976148488736162 0.5705877177071437 0.6447198332810333; visual box size=0.5976148488736162 0.5705877177071437 0.6447198332810333
- added link Link-z4, mass 1; collision box size=0.9588576729775992 0.6773770314593228 0.2618215354984731; visual box size=0.9588576729775992 0.6773770314593228 0.2618215354984731
- added link Link-z6, mass 1; collision box size=0.8418866241686216 0.861468927803236 0.21268672697202096; visual box size=0.8418866241686216 0.861468927803236 0.21268672697202096
- link Link-x0: geometry collision box size=0.2851538985695511 0.4894864188909096 0.4640608948981976; visual box size=0.2851538985695511 0.4894864188909096 0.4640608948981976
- link Link-y3: geometry collision box size=0.06571229089023056 0.10304916335464309 0.3476707195137332; visual box size=0.06571229089023056 0.10304916335464309 0.3476707195137332
Joints:
- removed joint Link-x0_Link-x1
- removed joint Link-x0_Link-y3
- removed joint Link-x0_Link-z2
- added joint Link-x0_Link-y1: type revolute, parent Link-x0, child Link-y1, origin xyz=0 0.2447432094454548 0.7053158690670012 rpy=0 0 0, axis 0 0 1, limit lower=-3.14159 upper=3.14159 effort=0.0 velocity=0.0
- added joint Link-x2_Link-y5: type revolute, parent Link-x2, child Link-y5, origin xyz=0 0.13256653590208017 0 rpy=0 0 0, axis 0 0 1, limit lower=-3.14159 upper=3.14159 effort=0.0 velocity=0.0
- added joint Link-x2_Link-z4: type revolute, parent Link-x2, child Link-z4, origin xyz=0 0 0.32785345816140116 rpy=0 0 0, axis 1 0 0, limit lower=-3.14159 upper=3.14159 effort=0.0 velocity=0.0
- added joint Link-y1_Link-x2: type revolute, parent Link-y1, child Link-x2, origin xyz=0.33378008374036694 0 0 rpy=0 0 0, axis 0 0 1, limit lower=-3.14159 upper=3.14159 effort=0.0 velocity=0.0
- added joint Link-y1_Link-y3: type revolute, parent Link-y1, child Link-y3, origin xyz=0 0.4829636587960703 0 rpy=0 0 0, axis 0 0 1, limit lower=-3.14159 upper=3.14159 effort=0.0 velocity=0.0
- added joint Link-z4_Link-z6: type revolute, parent Link-z4, child Link-z6, origin xyz=0 0 0.2618215354984731 rpy=0 0 0, axis 1 0 0, limit lower=-3.14159 upper=3.14159 effort=0.0 velocity=0.0
